Commit message: Add openduckpro2 robot package with URDF, meshes, and launch files
- Created CMakeLists.txt for building the openduckpro2 package.
- Added joint names configuration in YAML format.
- Implemented launch files for displaying the robot in RViz and simulating in Gazebo.
- Included STL mesh files for various robot components.
- Defined the robot's URDF model with detailed inertial and visual properties.
- Updated training script to reference openduckpro3 instead of openduckpro2.

File: resources/robots/openduckpro2/urdf/openduckpro2.urdf (robot description, URDF)
Before this commit: robot openduckpro2, 11 links, 10 joints
Links:
- link left_ankle_pitch_link: geometry collision mesh filename=../meshes/left_ankle_pitch_link.STL; visual mesh filename=../meshes/left_ankle_pitch_link.STL
- link right_ankle_pitch_link: geometry collision mesh filename=../meshes/right_ankle_pitch_link.STL; visual mesh filename=../meshes/right_ankle_pitch_link.STL
- link right_leg_yaw_link: mass 0.48200000 ->  0.48200000
Joints:
- joint left_ankle_pitch_joint: limit lower=-2 upper=2 effort=30 velocity=21 -> lower=-1 upper=1 effort=17 velocity=21
- joint left_knee_pitch_joint: limit lower=-2 upper=2 effort=30 velocity=21 -> lower=-1 upper=1 effort=17 velocity=21
- joint left_leg_pitch_joint: limit lower=-2 upper=2 effort=30 velocity=21 -> lower=-1 upper=1 effort=17 velocity=21
- joint left_leg_roll_joint: limit lower=-2 upper=2 effort=30 velocity=21 -> lower=-1 upper=1 effort=17 velocity=21
- joint left_leg_yaw_joint: limit lower=-2 upper=2 effort=30 velocity=21 -> lower=-1 upper=1 effort=17 velocity=21
- joint right_ankle_pitch_joint: limit lower=-2 upper=2 effort=30 velocity=21 -> lower=-1 upper=1 effort=17 velocity=21; origin xyz=0.10392 0.06 -0.0095 rpy=0 0 0 -> xyz=-0.10392 -0.06 -0.0095 rpy=0 0 -3.1416
- joint right_knee_pitch_joint: limit lower=-2 upper=2 effort=30 velocity=21 -> lower=-1 upper=1 effort=17 velocity=21; origin xyz=-0.06 0.10392 -0.0095 rpy=0 0 0 -> xyz=0.06 -0.10392 -0.0095 rpy=0 0 0
- joint right_leg_pitch_joint: limit lower=-2 upper=2 effort=30 velocity=21 -> lower=-1 upper=1 effort=17 velocity=21; origin xyz=0.0165 0 -0.049 rpy=0 -1.5708 0 -> xyz=-0.0165 0 -0.049 rpy=-1.5774 1.5708 -1.5775
- joint right_leg_roll_joint: limit lower=-2 upper=2 effort=30 velocity=21 -> lower=-1 upper=1 effort=17 velocity=21; origin xyz=0.00014573 -0.016499 -0.049 rpy=-1.5708 0 0.0088323 -> xyz=0 0.0165 -0.049 rpy=1.5708 0 0.00039951
- joint right_leg_yaw_joint: limit lower=-2 upper=2 effort=30 velocity=21 -> lower=-1 upper=1 effort=17 velocity=21; origin xyz=0 -0.075 -0.0005 rpy=0 0 -1.5666 -> xyz=0 -0.075 -0.0005 rpy=0 0 1.5666
