Commit message: [Fix] Track OpenDuckPro3 sole contact links

File: openduckpro3/urdf/openduckpro3.urdf (robot description, URDF)
Before this commit: robot openduckpro3, 12 links, 11 joints
Links:
- added link left_foot_link, mass 0.001; collision sphere radius=0.006; collision sphere radius=0.006
- added link right_foot_link, mass 0.001; collision sphere radius=0.006; collision sphere radius=0.006
- link left_ankle_pitch_link: geometry visual mesh filename=../meshes/right_ankle_pitch_link.STL
- link right_ankle_pitch_link: geometry visual mesh filename=../meshes/left_ankle_pitch_link.STL
Joints:
- added joint left_foot_fixed_joint: type fixed, parent left_ankle_pitch_link, child left_foot_link, origin xyz=-0.0004039554805933 -0.0610000009833932 -0.0154947293940548 rpy=0 0 0
- added joint right_foot_fixed_joint: type fixed, parent right_ankle_pitch_link, child right_foot_link, origin xyz=0 -0.061 0.0155 rpy=0 0 0
